Commit message: cleaned up description files

File: interbotix_descriptions/urdf/testing_environment.urdf.xacro (robot description, xacro)
@@ -23,33 +23,13 @@
   <!-- Call the init_widow_200 macro and give it the "arm B" namespace-->
   <xacro:init_widow_200 namespace="arm_B"/>
-  <!-- Create a prismatic joint between arm A and arm B (arm A will be the parent)-->
-  <!-- <xacro:macro name="arm_A_to_arm_B_joint" params="arm_A_robot_model arm_B_robot_model relative_x relative_y relative_z relative_roll relative_pitch relative_yaw">
-    <joint name="${arm_A_robot_model}_arm_A_to_${arm_B_robot_model}_arm_B" type="prismatic">
-      <parent link="${arm_A_robot_model}_arm_A/base_link"/>
-      <child link="${arm_B_robot_model}_arm_B/base_link"/>
-      <limit effort="1000.0" lower="0.01" upper="1.0" velocity="0.5"/>
-      <origin xyz="${relative_x} ${relative_y} ${relative_z}" rpy="${relative_roll} ${relative_pitch} ${relative_yaw}"/>
-      <axis xyz="0 1 0"/>
-    </joint>
-  </xacro:macro> -->
-  <!-- Call the macro for the prismatic joint between arm A and arm B -->
-  <!-- <xacro:arm_A_to_arm_B_joint arm_A_robot_model="$(arg arm_A_robot_model)" arm_B_robot_model="$(arg arm_B_robot_model)" relative_x="$(arg relative_x)" relative_y="$(arg relative_y)" relative_z="$(arg relative_z)" relative_roll="$(arg relative_roll)" relative_pitch="$(arg relative_pitch)" relative_yaw="$(arg relative_yaw)"/> -->
-  <!-- Add a world link before arm_A/base_link if using Moveit -->
-  <!-- <xacro:if value="$(arg moveit)">
-    <link name="world"/>
-    <joint name="world_to_arm_A_base_link" type="fixed">
-      <parent link="world"/>
-      <child link="$(arg arm_A_robot_model)_arm_A/base_link"/>
-    </joint>
-  </xacro:if> -->
   <!-- world link -->
-  <link name="world"/>
+  <!-- <link name="world"/> -->
   <!-- dummy link -->
   <link name="link0"/>
-  <joint name="world_joint" type="fixed">
+  <!-- <joint name="world_joint" type="fixed">
     <parent link="world"/>
     <child link="link0"/>
     <origin xyz="0 0 0" rpy="0 0 0"/>
-  </joint>
+  </joint> -->
   <!-- Arm A joint -->
   <joint name="link0_joint_arm_A" type="fixed">

Commit message: corrected launch files to take relative x,y,z and r,p,y between the arms from the testing_environment.launch command line args; had to make additions to move_group.launch and planning_context.launch

File: interbotix_descriptions/urdf/testing_environment.urdf.xacro (robot description, xacro)
@@ -1,7 +1,7 @@
 <?xml version="1.0"?>
 <robot name="testing_environment" xmlns:xacro="http://ros.org/wiki/xacro">
-  <xacro:arg name="robot_name" default = "testing_environment"/>
-  <xacro:arg name="arm_A_robot_model" default = "wx200"/>
-  <xacro:arg name="arm_B_robot_model" default = "wx200"/>
+  <xacro:arg name="robot_name" default="testing_environment"/>
+  <xacro:arg name="arm_A_robot_model" default="wx200"/>
+  <xacro:arg name="arm_B_robot_model" default="wx200"/>
   <xacro:arg name="default_gripper_bar" default="true"/>
   <xacro:arg name="default_gripper_fingers" default="true"/>
@@ -11,10 +11,10 @@
   <xacro:arg name="moveit" default="false"/>
   <!-- Relative displacement between arm A and arm B -->
-  <xacro:arg name="relative_x" default = "0"/>
-  <xacro:arg name="relative_y" default = "0.22"/>
-  <xacro:arg name="relative_z" default = "0"/>
-  <xacro:arg name="relative_roll" default = "0"/>
-  <xacro:arg name="relative_pitch" default = "0"/>
-  <xacro:arg name="relative_yaw" default = "0"/>
+  <xacro:arg name="relative_x" default=""/>
+  <xacro:arg name="relative_y" default=""/>
+  <xacro:arg name="relative_z" default=""/>
+  <xacro:arg name="relative_roll" default=""/>
+  <xacro:arg name="relative_pitch" default=""/>
+  <xacro:arg name="relative_yaw" default=""/>
   <!-- Importing Interbotix's URDF files for WidowX_200-->
   <xacro:include filename="$(find interbotix_descriptions)/urdf/wx200_modified.urdf.xacro"/>
@@ -42,5 +42,5 @@
     <parent link="link0"/>
     <child link="$(arg arm_B_robot_model)_arm_B/base_link"/>
-    <origin xyz="0 $(arg relative_y) 0" rpy="0 0 0"/>
+    <origin xyz="$(arg relative_x) $(arg relative_y) $(arg relative_z)" rpy="$(arg relative_roll) $(arg relative_pitch) $(arg relative_yaw)"/>
   </joint>
 </robot>
